File: pcb/CC40_ROM_Cart.sch (EAGLE design)
At the start: 15 parts, among them IC1 SST39SF040APH/27CXX(X), X1 EXPANSION_PORT_CC40_EDGE

Commit message: Updated layouts and measurements
Parts:
- added P1: CC40_CARTN, ti-cc40-74-95:CC40_CARTN
- IC1: value SST39SF040APH/27CXX(X) -> SST39SF040/27CXX(X); device memory-sst:SST39SF040APH -> memory-sst:SST39SF040APHR
- S1: device switch-dil:DP04 -> switch-dil-rp:DP04
- X1: value EXPANSION_PORT_CC40_EDGE -> EXPANSION_PORT_CC40; device ti-cc40:EXPANSION_PORT_CC40_EDGE -> ti-cc40-74-95:EXPANSION_PORT_CC40
Connections:
- net !CS: now also X1X.!CS_RAM, X1X.!CS_ROM; no longer X1X.!CS_CRAM, X1X.!CS_CROM
